File: kicad_sc11bbm/sc11bbm.kicad_sch (KiCad schematic)
At the start: 7 parts

Commit message: Update sc11bbm.kicad_sch
Parts:
- removed U?: QMC5883L, symbol QMC5883L:QMC5883L
- removed U?: ADXL335, symbol ADXL335:ADXL335
- added U?: QMC5883L, symbol QMC5883L:QMC5883L
- added U?: L3GD20H, symbol L3GD20H:L3GD20H
- added U?: ADXL335, symbol ADXL335:ADXL335
Connections:
- net at A?.13 (D10): now also U?.5 (CS)
- net at A?.14 (D11): now also U?.3 (SDA)
- net at A?.15 (D12): now also U?.4 (SA0)
- net at A?.16 (D13): now also U?.2 (SCL)
- net at A?.17 (3V3): now also U?.1 (+V), U?.1 (VCC)
- net at A?.23 (A4): now also U?.4 (SDA)
- net at A?.24 (A5): now also U?.3 (SCL), U?.4 (Z_out)
- net at A?.25 (A6): now also U?.3 (Y_out)
- net at A?.26 (A7): now also U?.2 (X_out)
- net at A?.27 (+5V): now also U?.1 (VCC)
- new net GND: U?.2 (GND), U?.5 (GND)
- no-connect marks 0 -> 1
Other:
- moved on the sheet: U?
