File: kicad_sc11bbm/sc11bbm.kicad_sch (KiCad schematic)
At the start: 8 parts

Commit message: Reference settings are not yet
Parts:
- removed U?: BME280, symbol BME280:BME280
- added M? (x2): Brushless motor, symbol Motor:Fan_3pin
- added Q?: 2SK4017, symbol Transistor_FET:2N7002E
- added RV?: NichromeWire, symbol Device:R_Potentiometer_US
- added U?: BMP280, symbol sc11bbm:BMP280
- added U? (x2): ESC, symbol sc11bbm:ESC
Connections:
- net +9V: now also RV?.2
- net GND: now also A?.29 (GND), A?.4 (GND), U?.1 (GND), U?.14 (GND), U?.2 (GND), U?.6 (VSS), U?.8 (GND), Q?.2 (S), U?. (Vin), U?. (Vin), U?.5 (GND)
- net D12: now reaches A?.15 (D12), U?.4 (SA0), U?.7 (DAT0)
- net D12: now also U?.1 (SDO)
- net D13: now reaches A?.16 (D13), U?.2 (SCL), U?.5 (CLK)
- net D13: now also U?.4 (SCL)
- net D11: now reaches A?.14 (D11), U?.3 (CMD), U?.3 (SDA)
- net D11: now also U?.3 (SDA)
- net D9: now reaches A?.12 (D9)
- net D9: now also U?.2 (CSB)
- net 3V3: now reaches A?.17 (3V3), U?.1 (+V), U?.1 (VCC), U?.4 (VDD)
- net 3V3: now also U?.28 (VCC), U?.6 (VCC)
- net 5V: now reaches U?.1 (5V)
- net 5V: now also A?.27 (+5V), U?.1 (VCC)
- net D3: now reaches U?.3 (RXD)
- net D3: now also A?.6 (D3)
- net D2: now reaches U?.4 (TXD)
- net D2: now also A?.5 (D2)
- net A5: now reaches A?.24 (A5), U?.3 (SCL)
- net A5: no longer U?.4 (Z_out)
- net A4: now reaches A?.23 (A4), U?.4 (SDA)
- net RX: now reaches U?.10 (DIO6/TX)
- net RX: now also A?.2 (D0/RX)
- net TX: now reaches U?.3 (DIO7/RX)
- net TX: now also A?.1 (D1/TX)
- net D10: now reaches A?.13 (D10), U?.5 (CS)
- net A0: now reaches A?.19 (A0)
- net A0: now also U?.4 (Z_out)
- net A1: now reaches A?.20 (A1)
- net A1: now also U?.3 (Y_out)
- net A2: now reaches A?.21 (A2)
- net A2: now also U?.2 (X_out)
- net at A?.25 (A6): no longer U?.3 (Y_out)
- net at A?.26 (A7): no longer U?.2 (X_out)
- net Lipo2: now reaches A?.30 (VIN)
- net D4: now reaches A?.7 (D4), U?.2 (CD/DAT3)
- net D4: now also U?. (Vin)
- net D5: now reaches A?.8 (D5)
- net D5: now also U?. (Vin)
- net D6: now reaches A?.9 (D6)
- net D6: now also Q?.1 (G)
- new net: Q?.3 (D), RV?.1
- new net: M?.1, U?. (Vin) (x2)
- new net: M?.2, U?. (Vin) (x2)
- new net: M?.3, U?. (Vin) (x2)
- new net Lipo3: U?. (Vin), U?. (Vin)
- no-connect marks 1 -> 0
Other:
- moved on the sheet: A?, U?

Commit message: Subtle changes to the schematic
Parts:
- removed U?: AE-GYSFDMAXB, symbol AE-GYSFDMAXB:AE-GYSFDMAXB
- removed U?: QMC5883L, symbol QMC5883L:QMC5883L
- removed U?: L3GD20H, symbol L3GD20H:L3GD20H
- removed U?: SD_CARD_DIP, symbol sc11bbm:SD_CARD_DIP
- removed U?: ADXL335, symbol ADXL335:ADXL335
- added U?: SD_CARD_DIP, symbol sc11bbm:SD_CARD_DIP
- added U?: AE-GYSFDMAXB, symbol sc11bbm:AE-GYSFDMAXB
- added U?: QMC5883L, symbol sc11bbm:QMC5883L
- added U?: L3GD20H, symbol sc11bbm:L3GD20H
- added U?: ADXL335, symbol sc11bbm:ADXL335
Connections:
- net 3V3: now also U?.1 (+V), U?.1 (VCC), U?.4 (VDD)
- net 5V: now also U?.1 (5V), U?.1 (VCC)
- net A0: now also U?.4 (Z_out)
- net A1: now also U?.3 (Y_out)
- net A2: now also U?.2 (X_out)
- net A4: now also U?.4 (SDA)
- net A5: now also U?.3 (SCL)
- net D10: now also U?.5 (CS)
- net D11: now also U?.3 (CMD), U?.3 (SDA)
- net D12: now also U?.4 (SA0), U?.7 (DAT0)
- net D13: now also U?.2 (SCL), U?.5 (CLK)
- net D2: now also U?.4 (TXD)
- net D3: now also U?.3 (RXD)
- net D4: now also U?.2 (CD/DAT3)
- net GND: now also U?.2 (GND), U?.2 (GND), U?.5 (GND), U?.6 (VSS), U?.8 (GND)
Other:
- moved on the sheet: M?, U?

Commit message: Circuit diagram completed
Parts:
- added BT1: Lipo2, sc11bbm:Lipo2, symbol Device:Battery_Cell
- added BT2: +9V, sc11bbm:power_9v, symbol Device:Battery_Cell
- added BT3: Lipo3, sc11bbm:Lipo3, symbol Device:Battery_Cell
- A1: renamed from A?; footprint Module:Arduino_Nano -> sc11bbm:Arduino_Nano
- M1: renamed from M?; value Brushless motor -> Brushless motor Right
- M2: renamed from M?; value Brushless motor -> Brushless motor Left
- Q1: renamed from Q?; footprint (none) -> sc11bbm:2SK4017
- RV1: renamed from RV?; footprint (none) -> sc11bbm:NichromeWire
- U1: renamed from U?; value ESC -> ESC_R; footprint (none) -> sc11bbm:ESC_R
- U2: renamed from U?; value ESC -> ESC_L; footprint (none) -> sc11bbm:ESC_L
- U4: renamed from U?; footprint (none) -> sc11bbm:QMC5883L
- U5: renamed from U?; footprint (none) -> sc11bbm:BMP280
- U7: renamed from U?; footprint (none) -> sc11bbm:AE-GYSFDMAXB
- U8: renamed from U?; footprint (none) -> sc11bbm:ADXL335
- U9: renamed from U?; footprint (none) -> sc11bbm:SD_CARD_DIP
- gave numbers to parts that had none: 2
Connections:
- net 3V3: now also U5.1 (VCC); no longer U5.6 (VCC)
- net D11: now also U5.4 (SDA); no longer U5.3 (SDA)
- net D12: now also U5.6 (SDO); no longer U5.1 (SDO)
- net D13: now also U5.3 (SCL); no longer U5.4 (SCL)
- net D4: now also U1.1 (PWM); no longer U1. (Vin)
- net D5: now also U2.1 (PWM); no longer U2. (Vin)
- net D9: now also U5.5 (CSB); no longer U5.2 (CSB)
- net GND: now also U1.3 (GND), U1.5 (GND), U2.3 (GND), U2.5 (GND), U5.2 (GND), BT1.2 (-), BT2.2 (-), BT3.2 (-); no longer U1. (Vin), U2. (Vin), U5.5 (GND)
- net Lipo2: now also BT1.1 (+)
- net Lipo3: now also U1.4 (Vin), U2.4 (Vin), BT3.1 (+); no longer U1. (Vin), U2. (Vin)
- net at M2.1: now also U2.6 (1); no longer U2. (Vin)
- net at M2.2: now also U2.7 (2); no longer U2. (Vin)
- net at M2.3: now also U2.8 (3); no longer U2. (Vin)
- net at M1.1: now also U1.6 (1); no longer U1. (Vin)
- net at M1.2: now also U1.7 (2); no longer U1. (Vin)
- net at M1.3: now also U1.8 (3); no longer U1. (Vin)
- net +9V: no longer names the net of RV1.2
- net +9V: now also BT2.1 (+)

Commit message: Order completed for Board ver1.0
Parts:
- U3: footprint (none) -> sc11bbm:L3GD20H
Connections:
- net GND: now also Q1.3 (S); no longer Q1.2 (S)
- net at RV1.1: now also Q1.2 (D); no longer Q1.3 (D)
Changed lines of the file:
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@@
   (symbol (lib_id "Transistor_FET:2N7002E") (at 66.04 85.09 270) (unit 1)
     (in_bom yes) (on_board yes) (fields_autoplaced)
-    (property "Reference" "Q1" (id 0) (at 66.04 92.71 90))
-    (property "Value" "2SK4017" (id 1) (at 66.04 95.25 90))
-    (property "Footprint" "sc11bbm:2SK4017" (id 2) (at 64.135 90.17 0)
+    (property "Reference" "Q1" (id 0) (at 58.42 85.09 90))
+    (property "Value" "2SK4017" (id 1) (at 55.88 85.09 90))
+    (property "Footprint" "sc11bbm:2SK4017" (id 2) (at 60.96 83.185 0)
       (effects (font (size 1.27 1.27) italic) (justify left) hide)
     )
@@
     (property "Reference" "U3" (id 0) (at 199.39 111.76 0))
     (property "Value" "L3GD20H" (id 1) (at 199.39 114.3 0))
-    (property "Footprint" "" (id 2) (at 199.39 114.3 0)
+    (property "Footprint" "sc11bbm:L3GD20H" (id 2) (at 199.39 114.3 0)
       (effects (font (size 1.27 1.27)) hide)
     )
@@
     )
     (path "/bce30d9d-5959-43c2-901a-216240c51ddc"
-      (reference "U3") (unit 1) (value "L3GD20H") (footprint "")
+      (reference "U3") (unit 1) (value "L3GD20H") (footprint "sc11bbm:L3GD20H")
     )
     (path "/40d8ad8c-b3b9-4b74-ac6c-a025ffa51987"

Commit message: For EM board2
Parts:
- added BT4: Lipo2, sc11bbm:Lipo2, symbol Device:Battery_Cell
- added BT5, BT6: Lipo3, sc11bbm:Lipo3, symbol Device:Battery_Cell
- added D1, D2, D3: LED, sc11bbm:LED, symbol Device:LED
- added R1, R2, R3: R, sc11bbm:Resistor, symbol pspice:R
- added SW1, SW2, SW3, SW4: SW_SPST, sc11bbm:swicth, symbol sc11bbm:SW_SPST
- added SW5: SW_SPST, sc11bbm:swicth, symbol Switch:SW_SPST
Connections:
- net GND: now also BT6.2 (-), D1.1 (K), D2.1 (K), D3.1 (K); no longer BT3.2 (-)
- net Lipo2: now also SW1.1 (A); no longer BT1.1 (+)
- net Lipo3: now also SW5.1 (A); no longer BT3.1 (+)
- net RX: now also SW2.1 (A); no longer A1.2 (D0/RX)
- net TX: now also SW3.1 (A); no longer A1.1 (D1/TX)
- net at RV1.2: now also SW4.1 (A); no longer BT2.1 (+)
- net D7: now reaches A1.10 (D7)
- net D7: now also R1.2
- net D8: now reaches A1.11 (D8)
- net D8: now also R2.2
- net A3: now reaches A1.22 (A3)
- net A3: now also R3.2
- new net: D1.2 (A), R1.1
- new net: BT3.2 (-), BT5.1 (+)
- new net: BT5.2 (-), BT6.1 (+)
- new net: D3.2 (A), R3.1
- new net: A1.1 (D1/TX), SW3.2 (B)
- new net: BT2.1 (+), SW4.2 (B)
- new net: BT3.1 (+), SW5.2 (B)
- new net: D2.2 (A), R2.1
- new net: BT4.1 (+), SW1.2 (B)
- new net: BT1.1 (+), BT4.2 (-)
- new net: A1.2 (D0/RX), SW2.2 (B)
Other:
- moved on the sheet: BT2, BT3
