File: kicad_sc11bbm/sc11bbm.kicad_pcb (KiCad board)
At the start: 2 copper layers, 100 x 100 mm, 21 parts, among them M1 MountingHole_3.2mm_M3_ISO14580, M2 MountingHole_3.2mm_M3_ISO14580, M3 MountingHole_3.2mm_M3_ISO14580, Q1 2SK4017, U1 ESC_R, U2 ESC_L, U3 L3GD20H, U4 QMC5883L, U5 BMP280, U6 MW-R-DP-W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

Commit message: For EM board2
Parts:
- removed the G*** at (212.3, 110.2)
- added BT3: Lipo3, sc11bbm:Lipo3, F.Cu at (223.7, 32.5)
- added BT4: Lipo2, sc11bbm:Lipo2, F.Cu at (168.0, 84.6)
- added BT5: Lipo3, sc11bbm:Lipo3, F.Cu at (230.0, 32.5)
- added BT6: Lipo3, sc11bbm:Lipo3, F.Cu at (217.5, 32.5)
- added C2: bighole, sc11bbm:bighole, F.Cu at (254.5, 65.5)
- added CI1: bighole, sc11bbm:bighole, F.Cu at (259.7, 77.2)
- added D1: LED, sc11bbm:LED, F.Cu at (193.5, 33.0)
- added D2: LED, sc11bbm:LED, F.Cu at (193.5, 29.5)
- added D3: LED, sc11bbm:LED, F.Cu at (193.5, 36.5)
- added G1: LOGO, sc11bbm:sc11logo2, B.Cu at (211.2, 116.0)
- added R1: R, sc11bbm:Resistor, F.Cu at (194.7, 47.2)
- added R2: R, sc11bbm:Resistor, F.Cu at (194.7, 40.2)
- added R3: R, sc11bbm:Resistor, F.Cu at (194.7, 43.8)
- added SW1: SW_SPST, sc11bbm:swicth, F.Cu at (185.5, 46.0)
- added SW2: SW_SPST, sc11bbm:swicth, F.Cu at (185.5, 41.5)
- added SW3: SW_SPST, sc11bbm:swicth, F.Cu at (185.5, 36.8)
- added SW4: SW_SPST, sc11bbm:swicth, F.Cu at (185.5, 50.5)
- added SW5: SW_SPST, sc11bbm:swicth, F.Cu at (237.5, 38.5)
- REF**, U8: moved to B.Cu
- moved G2 82.2 mm to (245.5, 47.2), turned to 90 degrees
- moved U4 64.1 mm to (238.8, 102.5)
- moved REF** 57.2 mm to (209.5, 83.5), turned to 0 degrees
- moved BT2 56.8 mm to (168.0, 85.9)
- moved U5 54.9 mm to (209.8, 44.9), turned to -90 degrees
- moved RV1 19.8 mm to (202.0, 26.2)
- moved U8 17.9 mm to (230.4, 69.8), turned to -90 degrees
- moved U1 12.5 mm to (168.0, 64.8), turned to 180 degrees
- moved U2 12.3 mm to (168.0, 71.6), turned to 180 degrees
- moved BT1 10.3 mm to (168.0, 78.1), turned to 180 degrees
- moved A1 5.07 mm to (180.6, 59.7)
- moved Q1 4.24 mm to (202.0, 34.0)
- moved U7 4.01 mm to (234.7, 69.5)
- moved G*** 3.71 mm to (213.5, 84.8)
- moved U3 2.92 mm to (225.5, 44.5), turned to 90 degrees
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- renumbered G*** to G2
Connections:
- A1 pad 1: TX -> Net-(A1-Pad1)
- A1 pad 10: unconnected-(A1-Pad10) -> D7
- A1 pad 11: unconnected-(A1-Pad11) -> D8
- A1 pad 2: RX -> Net-(A1-Pad2)
- A1 pad 22: unconnected-(A1-Pad22) -> A3
- BT1 pad 1: Lipo2 -> Net-(BT1-Pad1)
- RV1 pad 2: Net-(BT2-Pad1) -> Net-(RV1-Pad2)
Routing:
- net 5V: track 172.1 -> 68.2 mm
- net (no net): track 0.00 -> 75.7 mm, vias 0 -> 1
- net A2: track 42.9 -> 105.9 mm, vias 0 -> 1
- net 3V3: track 165.3 -> 102.8 mm, vias 1 -> 2
- net Lipo3: track 0.00 -> 60.1 mm
- net D8: track 0.00 -> 55.2 mm
- net Net-(RV1-Pad2): track 0.00 -> 49.5 mm
- net Net-(SW1-Pad2): track 0.00 -> 47.8 mm
- net D10: track 90.9 -> 136.7 mm
- net A3: track 0.00 -> 44.4 mm, vias 0 -> 1
- net Net-(BT2-Pad1): track 9.05 -> 52.3 mm
- net D7: track 0.00 -> 42.2 mm
- net Lipo2: track 58.2 -> 16.9 mm, vias 1 -> 0
- net GND: track 263.2 -> 301.1 mm, vias 7 -> 9
- net D13: track 120.4 -> 84.6 mm
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Other:
- board text added: "A3"
- board text added: "Board ver 2.0"
- board text added: "D7"
- board text added: "D8"
- board text added: "Lipo2"
- board text added: "Lipo3"
- board text added: "Nichr"
- board text added: "Note: Lipo3 circuit is connected by 1.1mm trace for auxiliary. Therefore, be sure to disconnect with the switch."
- board text added: "SC-11 Designed by Daisuke Nishihama"
- board text removed: "A3*"
- board text removed: "Board ver1.0"
- board text removed: "D7*"
- board text removed: "D8*"
- board text removed: "SC-11 Maked by Daisuke Nishihama"
